File: design/KIRB/LP_MSPM0G3507_HDR.kicad_sch (KiCad schematic)
At the start: 33 parts, among them J2 J_IN1/J_IN3, J3 J_IN4/J_IN2, J4 USB_B_Micro

Commit message: started ult software
Parts:
- renumbered C7 to C2, J2 to J1, J3 to J2, J4 to J3, R22 to R10, R23 to R11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
