File: design/KIRB/LP_MSPM0G3507_HDR.kicad_sch (KiCad schematic)
At the start: 33 parts, among them J1 J_IN1/J_IN3, J2 J_IN4/J_IN2, J3 USB_B_Micro

Commit message: added kirb3 graphic
Parts:
- added R36: 0 Ω, symbol Device:R_US
Connections:
- net at J2.35 (PB13): now also R36.2
- net PING_IO renamed ECHO
- new net TRIG: R36.1
- no-connect marks 11 -> 10
Changed lines of the file:
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@@
-	)
-	(no_connect
-		(at 165.1 72.39)
 	)
 	(no_connect
@@
 	(wire
 		(pts
-			(xy 165.1 72.39) (xy 167.64 72.39)
+			(xy 156.21 72.39) (xy 160.02 72.39)
 		)
 		(stroke
@@
 	(wire
 		(pts
-			(xy 165.1 91.44) (xy 167.64 91.44)
+			(xy 157.48 91.44) (xy 167.64 91.44)
 		)
 		(stroke
@@
 		)
 	)
+	(hierarchical_label "TRIG"
+		(shape bidirectional)
+		(at 156.21 72.39 180)
+		(effects
+			(font
+				(size 1.27 1.27)
+			)
+			(justify right)
+		)
+	)
 	(hierarchical_label "PWM_MTR[1..2]"
 		(shape output)
@@
 		)
 	)
-	(hierarchical_label "PING_IO"
+	(hierarchical_label "ECHO"
 		(shape bidirectional)
-		(at 165.1 91.44 180)
+		(at 157.48 91.44 180)
 		(effects
 			(font
@@
 					(unit 1)
 				)
+			)
+		)
+	)
+	(symbol
+		(lib_id "Device:R_US")
+		(at 163.83 72.39 90)
+		(unit 1)
+		(exclude_from_sim no)
+		(in_bom yes)
+		(on_board yes)
+		(dnp no)
+		(property "Reference" "R36"
+			(at 163.83 68.58 90)
+			(effects
+				(font
+					(size 1.27 1.27)
+				)
+			)
+		)
+		(property "Value" "0 Ω"
+			(at 163.83 70.358 90)
+			(effects
+				(font
+					(size 1.27 1.27)
+				)
+			)
+		)
+		(property "Footprint" ""
+			(at 164.084 71.374 90)
+			(effects
+				(font
+					(size 1.27 1.27)
+				)
+				(hide yes)
+			)
+		)
+		(property "Datasheet" "~"
+			(at 163.83 72.39 0)
+			(effects
+				(font
+					(size 1.27 1.27)
+				)
+				(hide yes)
+			)
+		)
+		(property "Description" "Resistor, US symbol"
+			(at 163.83 72.39 0)
+			(effects
+				(font
+					(size 1.27 1.27)
+				)
+				(hide yes)
+			)
+		)
+		(pin "1"
+		)
+		(pin "2"
+		)
+		(instances
+			(project "KIRB"
+				(path "/0a51f53b-36a2-49a0-b5b8-e2ed0cb11e2a/f7853a98-918c-411e-85ae-dd3031adf4af"
+					(reference "R36")
+					(unit 1)
+				)

Commit message: remove obsolete files
Other:
- title: LP-MSPM0G3507 Headers -> Kinematic Intelligent Ranging Bot (KIRB-3)
Changed lines of the file:
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@@
 	(paper "USLetter")
 	(title_block
-		(title "LP-MSPM0G3507 Headers")
+		(title "Kinematic Intelligent Ranging Bot (KIRB-3)")
 		(date "2025-11-30")
 	)
