File: design/KIRB/ULTRASONICS.kicad_sch (KiCad schematic)
At the start: 13 parts, among them U2 PING, U3 PING, U4 SN74LVC245A, U5 PING, U6 PING, U7 74HC4051, U8 74HC4051

Commit message: started ult software
Parts:
- removed U2, U3, U5, U6: PING, symbol Connector_Generic:Conn_01x03
- added U11, U12, U13, U14, U15, U16, U17, U18, U19, U20: PING, symbol Connector_Generic:Conn_01x03
- renumbered C3 to C6, C4 to C7, R4 to R33, R3 to R34, R5 to R35, U8 to U10, U7 to U8, U4 to U9
Connections:
- net +5V: now also U11.2 (+5V), U12.2 (+5V), U13.2 (+5V), U14.2 (+5V), U15.2 (+5V), U16.2 (+5V), U17.2 (+5V), U18.2 (+5V), U19.2 (+5V), U20.2 (+5V)
- net GND: now also U11.1 (GND), U12.1 (GND), U13.1 (GND), U14.1 (GND), U15.1 (GND), U16.1 (GND), U17.1 (GND), U18.1 (GND), U19.1 (GND), U20.1 (GND)
- net PING0: now also U11.3 (SIG)
- net PING1: now also U12.3 (SIG)
- net PING2: now also U13.3 (SIG)
- net PING3: now also U14.3 (SIG)
- net PING4: now also U15.3 (SIG)
- net PING5: now also U16.3 (SIG)
- net PING6: now also U17.3 (SIG)
- net PING7: now also U18.3 (SIG)
- net PING8: now also U19.3 (SIG)
- net PING9: now also U20.3 (SIG)
Other:
- note removed: "..."
- moved on the sheet: C5, C6, C7, R33, R34, R35, U10, U8, U9
