File: design/KIRB/ULTRASONICS.kicad_sch (KiCad schematic)
At the start: 19 parts, among them U10 74HC4051, U11 PING, U12 PING, U13 PING, U14 PING, U15 PING, U16 PING, U17 PING, U18 PING, U19 PING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

Commit message: remove obsolete files
Other:
- title: Ultrasonic Sensing System -> Kinematic Intelligent Ranging Bot (KIRB-3)
Changed lines of the file:
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@@
 	(generator "eeschema")
 	(generator_version "9.0")
-	(paper "A4")
+	(paper "USLetter")
 	(title_block
-		(title "Ultrasonic Sensing System")
+		(title "Kinematic Intelligent Ranging Bot (KIRB-3)")
 		(date "2025-12-01")
 	)
