File: design/KIRB/MOTOR_IF.kicad_sch (KiCad schematic)
At the start: 6 parts, among them U15 HB25 Motor Controller, U16 HB25 Motor Controller, U17 36-Pos Quadrature Encoder, U18 36-Pos Quadrature Encoder

Commit message: started ult software
Parts:
- gave numbers to parts that had none: 2
- renumbered U15 to U4, U16 to U5, U17 to U6, U18 to U7
Changed lines of the file:
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@@
 		(on_board yes)
 		(dnp no)
-		(property "Reference" "#PWR040"
+		(property "Reference" "#PWR027"
 			(at 83.82 96.52 0)
 			(effects
@@
 			(project "KIRB"
 				(path "/0a51f53b-36a2-49a0-b5b8-e2ed0cb11e2a/e9b55cd3-e9fe-4149-ac8f-4fb25ab6db08"
-					(reference "#PWR040")
+					(reference "#PWR027")
 					(unit 1)
 				)
@@
 		(on_board yes)
 		(dnp no)
-		(property "Reference" "U15"
+		(property "Reference" "U4"
 			(at 107.95 72.644 0)
 			(effects
@@
 			(project "KIRB"
 				(path "/0a51f53b-36a2-49a0-b5b8-e2ed0cb11e2a/e9b55cd3-e9fe-4149-ac8f-4fb25ab6db08"
-					(reference "U15")
+					(reference "U4")
 					(unit 1)
 				)
@@
 		(on_board yes)
 		(dnp no)
-		(property "Reference" "#PWR057"
+		(property "Reference" "#PWR028"
 			(at 144.78 96.52 0)
 			(effects
@@
 			(project "KIRB"
 				(path "/0a51f53b-36a2-49a0-b5b8-e2ed0cb11e2a/e9b55cd3-e9fe-4149-ac8f-4fb25ab6db08"
-					(reference "#PWR057")
+					(reference "#PWR028")
 					(unit 1)
 				)
@@
 		(dnp no)
 		(fields_autoplaced yes)
-		(property "Reference" "M?"
+		(property "Reference" "M2"
 			(at 190.5 86.3599 0)
 			(effects
@@
 			(project ""
 				(path "/0a51f53b-36a2-49a0-b5b8-e2ed0cb11e2a/e9b55cd3-e9fe-4149-ac8f-4fb25ab6db08"
-					(reference "M?")
+					(reference "M2")
 					(unit 1)
 				)
@@
 		(on_board yes)
 		(dnp no)
-		(property "Reference" "#PWR059"
+		(property "Reference" "#PWR026"
 			(at 153.67 78.74 0)
 			(effects
@@
 			(project "KIRB"
 				(path "/0a51f53b-36a2-49a0-b5b8-e2ed0cb11e2a/e9b55cd3-e9fe-4149-ac8f-4fb25ab6db08"
-					(reference "#PWR059")
+					(reference "#PWR026")
 					(unit 1)
 				)
@@
 		(dnp no)
 		(fields_autoplaced yes)
-		(property "Reference" "U17"
+		(property "Reference" "U6"
 			(at 109.474 120.904 0)
 			(effects
@@
 			(project "KIRB"
 				(path "/0a51f53b-36a2-49a0-b5b8-e2ed0cb11e2a/e9b55cd3-e9fe-4149-ac8f-4fb25ab6db08"
-					(reference "U17")
+					(reference "U6")
 					(unit 1)
 				)
@@
 		(on_board yes)
 		(dnp no)
-		(property "Reference" "#PWR062"
+		(property "Reference" "#PWR030"
 			(at 185.42 127 0)
 			(effects
@@
 			(project "KIRB"
 				(path "/0a51f53b-36a2-49a0-b5b8-e2ed0cb11e2a/e9b55cd3-e9fe-4149-ac8f-4fb25ab6db08"
-					(reference "#PWR062")
+					(reference "#PWR030")
 					(unit 1)
 				)
@@
 		(on_board yes)
 		(dnp no)
-		(property "Reference" "U16"
+		(property "Reference" "U5"
 			(at 168.91 72.644 0)
 			(effects
@@
 			(project "KIRB"
 				(path "/0a51f53b-36a2-49a0-b5b8-e2ed0cb11e2a/e9b55cd3-e9fe-4149-ac8f-4fb25ab6db08"
-					(reference "U16")
+					(reference "U5")
 					(unit 1)
 				)
@@
 		(on_board yes)
 		(dnp no)
-		(property "Reference" "#PWR063"
+		(property "Reference" "#PWR032"
 			(at 185.42 139.7 0)
 			(effects
@@
 			(project "KIRB"
 				(path "/0a51f53b-36a2-49a0-b5b8-e2ed0cb11e2a/e9b55cd3-e9fe-4149-ac8f-4fb25ab6db08"
-					(reference "#PWR063")
+					(reference "#PWR032")
 					(unit 1)
 				)
@@
 		(dnp no)
 		(fields_autoplaced yes)
-		(property "Reference" "U18"
+		(property "Reference" "U7"
 			(at 162.814 120.904 0)
 			(effects
@@
 			(project "KIRB"
 				(path "/0a51f53b-36a2-49a0-b5b8-e2ed0cb11e2a/e9b55cd3-e9fe-4149-ac8f-4fb25ab6db08"
-					(reference "U18")
+					(reference "U7")
 					(unit 1)
 				)
@@
 		(on_board yes)
 		(dnp no)
-		(property "Reference" "#PWR060"
+		(property "Reference" "#PWR029"
 			(at 132.08 127 0)
 			(effects
@@
 			(project "KIRB"
 				(path "/0a51f53b-36a2-49a0-b5b8-e2ed0cb11e2a/e9b55cd3-e9fe-4149-ac8f-4fb25ab6db08"
-					(reference "#PWR060")
+					(reference "#PWR029")
 					(unit 1)
 				)
@@
 		(on_board yes)
 		(dnp no)
-		(property "Reference" "#PWR058"
+		(property "Reference" "#PWR025"
 			(at 92.71 78.74 0)
 			(effects
@@
 			(project "KIRB"
 				(path "/0a51f53b-36a2-49a0-b5b8-e2ed0cb11e2a/e9b55cd3-e9fe-4149-ac8f-4fb25ab6db08"
-					(reference "#PWR058")
+					(reference "#PWR025")
 					(unit 1)
 				)
@@
 		(on_board yes)
 		(dnp no)
-		(property "Reference" "#PWR061"
+		(property "Reference" "#PWR031"
 			(at 132.08 139.7 0)
 			(effects
@@
 			(project "KIRB"
 				(path "/0a51f53b-36a2-49a0-b5b8-e2ed0cb11e2a/e9b55cd3-e9fe-4149-ac8f-4fb25ab6db08"
-					(reference "#PWR061")
+					(reference "#PWR031")
 					(unit 1)
 				)
@@
 		(dnp no)
 		(fields_autoplaced yes)
-		(property "Reference" "M?"
+		(property "Reference" "M1"
 			(at 129.54 86.3599 0)
 			(effects
@@
 			(project ""
 				(path "/0a51f53b-36a2-49a0-b5b8-e2ed0cb11e2a/e9b55cd3-e9fe-4149-ac8f-4fb25ab6db08"
-					(reference "M?")
-					(unit 1)
-				)
+					(reference "M1")
+					(unit 1)
+				)

Commit message: remove obsolete files
Other:
- title: Motor Drive System -> Kinematic Intelligent Ranging Bot (KIRB-3)
Changed lines of the file:
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@@
 	(paper "USLetter")
 	(title_block
-		(title "Motor Drive System")
+		(title "Kinematic Intelligent Ranging Bot (KIRB-3)")
 	)
 	(rectangle
