File: design/KIRB/POWER.kicad_sch (KiCad schematic)
At the start: 10 parts, among them J1 3S Balance Connector, SW1 Power Switch, U1 DC-DC Buck Converter Module

Commit message: started ult software
Parts:
- renumbered C1 to C3, C2 to C4, J1 to J4, R1 to R31, R2 to R32, U1 to U3
Changed lines of the file:
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@@
 		(on_board yes)
 		(dnp no)
-		(property "Reference" "#PWR06"
+		(property "Reference" "#PWR021"
 			(at 129.54 87.63 0)
 			(effects
@@
 			(project "KIRB"
 				(path "/0a51f53b-36a2-49a0-b5b8-e2ed0cb11e2a/024070e9-0b5c-4a13-970d-8a980a45ce1f"
-					(reference "#PWR06")
+					(reference "#PWR021")
 					(unit 1)
 				)
@@
 		(on_board yes)
 		(dnp no)
-		(property "Reference" "#PWR03"
+		(property "Reference" "#PWR019"
 			(at 214.63 69.85 0)
 			(effects
@@
 			(project "KIRB"
 				(path "/0a51f53b-36a2-49a0-b5b8-e2ed0cb11e2a/024070e9-0b5c-4a13-970d-8a980a45ce1f"
-					(reference "#PWR03")
+					(reference "#PWR019")
 					(unit 1)
 				)
@@
 		(on_board yes)
 		(dnp no)
-		(property "Reference" "#PWR05"
+		(property "Reference" "#PWR020"
 			(at 78.74 87.63 0)
 			(effects
@@
 			(project "KIRB"
 				(path "/0a51f53b-36a2-49a0-b5b8-e2ed0cb11e2a/024070e9-0b5c-4a13-970d-8a980a45ce1f"
-					(reference "#PWR05")
+					(reference "#PWR020")
 					(unit 1)
 				)
@@
 		(on_board yes)
 		(dnp no)
-		(property "Reference" "C2"
+		(property "Reference" "C4"
 			(at 203.454 66.294 0)
 			(effects
@@
 			(project "KIRB"
 				(path "/0a51f53b-36a2-49a0-b5b8-e2ed0cb11e2a/024070e9-0b5c-4a13-970d-8a980a45ce1f"
-					(reference "C2")
+					(reference "C4")
 					(unit 1)
 				)
@@
 		(on_board yes)
 		(dnp no)
-		(property "Reference" "#PWR01"
+		(property "Reference" "#PWR017"
 			(at 78.74 69.85 0)
 			(effects
@@
 			(project "KIRB"
 				(path "/0a51f53b-36a2-49a0-b5b8-e2ed0cb11e2a/024070e9-0b5c-4a13-970d-8a980a45ce1f"
-					(reference "#PWR01")
+					(reference "#PWR017")
 					(unit 1)
 				)
@@
 		(on_board yes)
 		(dnp no)
-		(property "Reference" "U1"
+		(property "Reference" "U3"
 			(at 168.91 66.04 0)
 			(effects
@@
 			(project "KIRB"
 				(path "/0a51f53b-36a2-49a0-b5b8-e2ed0cb11e2a/024070e9-0b5c-4a13-970d-8a980a45ce1f"
-					(reference "U1")
+					(reference "U3")
 					(unit 1)
 				)
@@
 		(on_board yes)
 		(dnp no)
-		(property "Reference" "#PWR07"
+		(property "Reference" "#PWR022"
 			(at 214.63 87.63 0)
 			(effects
@@
 			(project "KIRB"
 				(path "/0a51f53b-36a2-49a0-b5b8-e2ed0cb11e2a/024070e9-0b5c-4a13-970d-8a980a45ce1f"
-					(reference "#PWR07")
+					(reference "#PWR022")
 					(unit 1)
 				)
@@
 		(dnp no)
 		(fields_autoplaced yes)
-		(property "Reference" "R2"
+		(property "Reference" "R32"
 			(at 146.05 123.1899 0)
 			(effects
@@
 			(project "KIRB"
 				(path "/0a51f53b-36a2-49a0-b5b8-e2ed0cb11e2a/024070e9-0b5c-4a13-970d-8a980a45ce1f"
-					(reference "R2")
+					(reference "R32")
 					(unit 1)
 				)
@@
 		(on_board yes)
 		(dnp no)
-		(property "Reference" "#PWR04"
+		(property "Reference" "#PWR023"
 			(at 128.27 120.65 0)
 			(effects
@@
 			(project "KIRB"
 				(path "/0a51f53b-36a2-49a0-b5b8-e2ed0cb11e2a/024070e9-0b5c-4a13-970d-8a980a45ce1f"
-					(reference "#PWR04")
+					(reference "#PWR023")
 					(unit 1)
 				)
@@
 		(on_board yes)
 		(dnp no)
-		(property "Reference" "C1"
+		(property "Reference" "C3"
 			(at 190.754 66.04 0)
 			(effects
@@
 			(project "KIRB"
 				(path "/0a51f53b-36a2-49a0-b5b8-e2ed0cb11e2a/024070e9-0b5c-4a13-970d-8a980a45ce1f"
-					(reference "C1")
+					(reference "C3")
 					(unit 1)
 				)
@@
 		(on_board yes)
 		(dnp no)
-		(property "Reference" "#PWR08"
+		(property "Reference" "#PWR024"
 			(at 143.51 138.43 0)
 			(effects
@@
 			(project "KIRB"
 				(path "/0a51f53b-36a2-49a0-b5b8-e2ed0cb11e2a/024070e9-0b5c-4a13-970d-8a980a45ce1f"
-					(reference "#PWR08")
+					(reference "#PWR024")
 					(unit 1)
 				)
@@
 		(dnp no)
 		(fields_autoplaced yes)
-		(property "Reference" "J1"
+		(property "Reference" "J4"
 			(at 113.665 115.57 0)
 			(effects
@@
 			(project "KIRB"
 				(path "/0a51f53b-36a2-49a0-b5b8-e2ed0cb11e2a/024070e9-0b5c-4a13-970d-8a980a45ce1f"
-					(reference "J1")
+					(reference "J4")
 					(unit 1)
 				)
@@
 		(on_board yes)
 		(dnp no)
-		(property "Reference" "#PWR02"
+		(property "Reference" "#PWR018"
 			(at 129.54 69.85 0)
 			(effects
@@
 			(project "KIRB"
 				(path "/0a51f53b-36a2-49a0-b5b8-e2ed0cb11e2a/024070e9-0b5c-4a13-970d-8a980a45ce1f"
-					(reference "#PWR02")
+					(reference "#PWR018")
 					(unit 1)
 				)
@@
 		(on_board yes)
 		(dnp no)
-		(property "Reference" "R1"
+		(property "Reference" "R31"
 			(at 138.43 116.586 90)
 			(effects
@@
 			(project "KIRB"
 				(path "/0a51f53b-36a2-49a0-b5b8-e2ed0cb11e2a/024070e9-0b5c-4a13-970d-8a980a45ce1f"
-					(reference "R1")
-					(unit 1)
-				)
+					(reference "R31")
+					(unit 1)
+				)

Commit message: remove obsolete files
Other:
- title: Power Distribution System -> Kinematic Intelligent Ranging Bot (KIRB-3)
Changed lines of the file:
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@@
 	(paper "USLetter")
 	(title_block
-		(title "Power Distribution System")
+		(title "Kinematic Intelligent Ranging Bot (KIRB-3)")
 	)
 	(rectangle
