File: design/KIRB/RC_RECV_IF.kicad_sch (KiCad schematic)
At the start: 4 parts, among them U13 FS-iA6B, U14 SN74LVC245A

Commit message: started ult software
Parts:
- renumbered C6 to C1, R13 to R1, U13 to U1, U14 to U2
Changed lines of the file:
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@@
 		(on_board yes)
 		(dnp no)
-		(property "Reference" "#PWR043"
+		(property "Reference" "#PWR04"
 			(at 116.84 83.82 0)
 			(effects
@@
 			(project "KIRB"
 				(path "/0a51f53b-36a2-49a0-b5b8-e2ed0cb11e2a/b22f0d18-4d91-4b8e-a8f8-7677d2a7d09e"
-					(reference "#PWR043")
+					(reference "#PWR04")
 					(unit 1)
 				)
@@
 		(on_board yes)
 		(dnp no)
-		(property "Reference" "#PWR045"
+		(property "Reference" "#PWR01"
 			(at 134.62 68.58 0)
 			(effects
@@
 			(project "KIRB"
 				(path "/0a51f53b-36a2-49a0-b5b8-e2ed0cb11e2a/b22f0d18-4d91-4b8e-a8f8-7677d2a7d09e"
-					(reference "#PWR045")
+					(reference "#PWR01")
 					(unit 1)
 				)
@@
 		(on_board yes)
 		(dnp no)
-		(property "Reference" "#PWR044"
+		(property "Reference" "#PWR02"
 			(at 121.92 74.93 0)
 			(effects
@@
 			(project "KIRB"
 				(path "/0a51f53b-36a2-49a0-b5b8-e2ed0cb11e2a/b22f0d18-4d91-4b8e-a8f8-7677d2a7d09e"
-					(reference "#PWR044")
+					(reference "#PWR02")
 					(unit 1)
 				)
@@
 		(on_board yes)
 		(dnp no)
-		(property "Reference" "U13"
+		(property "Reference" "U1"
 			(at 82.55 76.708 0)
 			(effects
@@
 			(project "KIRB"
 				(path "/0a51f53b-36a2-49a0-b5b8-e2ed0cb11e2a/b22f0d18-4d91-4b8e-a8f8-7677d2a7d09e"
-					(reference "U13")
+					(reference "U1")
 					(unit 1)
 				)
@@
 		(on_board yes)
 		(dnp no)
-		(property "Reference" "#PWR042"
+		(property "Reference" "#PWR06"
 			(at 99.06 85.09 0)
 			(effects
@@
 			(project "KIRB"
 				(path "/0a51f53b-36a2-49a0-b5b8-e2ed0cb11e2a/b22f0d18-4d91-4b8e-a8f8-7677d2a7d09e"
-					(reference "#PWR042")
+					(reference "#PWR06")
 					(unit 1)
 				)
@@
 		(on_board yes)
 		(dnp no)
-		(property "Reference" "C6"
+		(property "Reference" "C1"
 			(at 128.016 61.214 90)
 			(effects
@@
 			(project "KIRB"
 				(path "/0a51f53b-36a2-49a0-b5b8-e2ed0cb11e2a/b22f0d18-4d91-4b8e-a8f8-7677d2a7d09e"
-					(reference "C6")
+					(reference "C1")
 					(unit 1)
 				)
@@
 		(on_board yes)
 		(dnp no)
-		(property "Reference" "#PWR041"
+		(property "Reference" "#PWR03"
 			(at 92.71 77.47 0)
 			(effects
@@
 			(project "KIRB"
 				(path "/0a51f53b-36a2-49a0-b5b8-e2ed0cb11e2a/b22f0d18-4d91-4b8e-a8f8-7677d2a7d09e"
-					(reference "#PWR041")
+					(reference "#PWR03")
 					(unit 1)
 				)
@@
 		(on_board yes)
 		(dnp no)
-		(property "Reference" "#PWR047"
+		(property "Reference" "#PWR05"
 			(at 152.4 90.17 0)
 			(effects
@@
 			(project "KIRB"
 				(path "/0a51f53b-36a2-49a0-b5b8-e2ed0cb11e2a/b22f0d18-4d91-4b8e-a8f8-7677d2a7d09e"
-					(reference "#PWR047")
+					(reference "#PWR05")
 					(unit 1)
 				)
@@
 		(on_board yes)
 		(dnp no)
-		(property "Reference" "U14"
+		(property "Reference" "U2"
 			(at 137.16 73.406 0)
 			(effects
@@
 			(project "KIRB"
 				(path "/0a51f53b-36a2-49a0-b5b8-e2ed0cb11e2a/b22f0d18-4d91-4b8e-a8f8-7677d2a7d09e"
-					(reference "U14")
+					(reference "U2")
 					(unit 1)
 				)
@@
 		(on_board yes)
 		(dnp no)
-		(property "Reference" "R13"
+		(property "Reference" "R1"
 			(at 128.27 112.268 90)
 			(effects
@@
 			(project "KIRB"
 				(path "/0a51f53b-36a2-49a0-b5b8-e2ed0cb11e2a/b22f0d18-4d91-4b8e-a8f8-7677d2a7d09e"
-					(reference "R13")
+					(reference "R1")
 					(unit 1)
 				)
@@
 		(on_board yes)
 		(dnp no)
-		(property "Reference" "#PWR046"
+		(property "Reference" "#PWR07"
 			(at 134.62 128.27 0)
 			(effects
@@
 			(project "KIRB"
 				(path "/0a51f53b-36a2-49a0-b5b8-e2ed0cb11e2a/b22f0d18-4d91-4b8e-a8f8-7677d2a7d09e"
-					(reference "#PWR046")
-					(unit 1)
-				)
+					(reference "#PWR07")
+					(unit 1)
+				)

Commit message: remove obsolete files
Other:
- title: RC Reciever Interface -> Kinematic Intelligent Ranging Bot (KIRB-3)
Changed lines of the file:
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@@
 	(paper "USLetter")
 	(title_block
-		(title "RC Reciever Interface")
+		(title "Kinematic Intelligent Ranging Bot (KIRB-3)")
 		(date "2025-11-30")
 	)
